File: IMU_Haptic_Audio_Display.kicad_sch (KiCad schematic)
At the start: 28 parts, among them J2 Conn_01x02, J3 Conn_01x13, J4 Conn_01x02, U3 DRV2603, U4 LSM6DSOX, U5 REG710NA-3.3/250, U6 SGTL5000

Commit message: Ref link added & Removed charge pumps
Parts:
- removed C17, C19: 4.7uF, Capacitor_SMD:C_0402_1005Metric, symbol Device:C
- removed C18: 0.22uF, Capacitor_SMD:C_0402_1005Metric, symbol Device:C
- removed U5: REG710NA-3.3/250, Package_TO_SOT_SMD:SOT-23-6, symbol Custom_Libs:REG710xx
Connections:
- net DISP_3.3V is gone; now on net MCU_3.3V: J3.1 (Pin_1)
