File: wifi.kicad_sch (KiCad schematic)
At the start: 37 parts, among them U8 NRF7002-QFAA-R, U9 DPX1608LKF3R2460A, Y3 40 MHz

Commit message: updated version
Parts:
- C64, C65: value 22nF -> 12pF
Other:
- note added: "1) 8-54 MHz crystal oscillator with load capacitance (C_L) = 8 pF"
